File: project/AllegroCurrentSensor/AllegroCurrentSensor.kicad_pcb (KiCad board)
At the start: 2 copper layers, 40 x 40 mm, 19 parts, among them J1 Conn_01x01_Female, J2 Conn_01x01_Female, J3 Conn_01x03_Female, U1 ACS713xLCTR-20A, U2 AD8651

Commit message: 発注用データ作成
Parts:
- moved H1 0.28 mm to (63.5, 66.5)
- moved H2 0.28 mm to (63.5, 33.5)
Other:
- board text added: "1"
- board text added: "3"
- board text added: "5V"
- board text added: "CS"
- board text added: "Current sensor v1.0-Allegro"
- board text added: "GND"
- board text added: "Vout"
Changed lines of the file:
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@@
   (general
     (thickness 1.6)
-    (drawings 6)
+    (drawings 21)
     (tracks 59)
     (zones 0)
@@
     (pad_drill 0.6)
     (pad_to_mask_clearance 0)
+    (solder_mask_min_width 0.25)
     (aux_axis_origin 0 0)
-    (visible_elements FFFFFF7F)
+    (visible_elements 7FFFFFFF)
     (pcbplotparams
       (layerselection 0x010fc_ffffffff)
@@
     (tags "capacitor handsolder")
     (attr smd)
-    (fp_text reference C1 (at 0 -1.43 180) (layer F.SilkS)
+    (fp_text reference C1 (at -2.6675 0 180) (layer F.SilkS)
       (effects (font (size 1 1) (thickness 0.15)))
     )
@@
     (tags "capacitor handsolder")
     (attr smd)
-    (fp_text reference C3 (at 0 -1.43) (layer F.SilkS)
+    (fp_text reference C3 (at 2.9525 0.02) (layer F.SilkS)
       (effects (font (size 1 1) (thickness 0.15)))
     )
@@
   )
   (module MountingHole:MountingHole_3.2mm_M3 (layer F.Cu)
-    (at 63.3 66.7)
+    (at 63.5 66.5)
     (descr "Mounting Hole 3.2mm, no annular, M3")
     (tags "mounting hole 3.2mm no annular m3")
     (attr virtual)
-    (fp_text reference H1 (at 0 -4.2) (layer F.SilkS)
+    (fp_text reference H1 (at 0 -4.2) (layer F.SilkS) hide
       (effects (font (size 1 1) (thickness 0.15)))
     )
@@
   )
   (module MountingHole:MountingHole_3.2mm_M3 (layer F.Cu)
-    (at 63.3 33.3)
+    (at 63.5 33.5)
     (descr "Mounting Hole 3.2mm, no annular, M3")
     (tags "mounting hole 3.2mm no annular m3")
     (attr virtual)
-    (fp_text reference H2 (at 0 -4.2) (layer F.SilkS)
+    (fp_text reference H2 (at 0 -4.2) (layer F.SilkS) hide
       (effects (font (size 1 1) (thickness 0.15)))
     )
@@
     (tags "mounting hole 3.2mm no annular m3")
     (attr virtual)
-    (fp_text reference H3 (at 0 -4.2) (layer F.SilkS)
+    (fp_text reference H3 (at 0 -4.2) (layer F.SilkS) hide
       (effects (font (size 1 1) (thickness 0.15)))
     )
@@
     (tags "mounting hole 3.2mm no annular m3")
     (attr virtual)
-    (fp_text reference H4 (at 0 -4.2) (layer F.SilkS)
+    (fp_text reference H4 (at 0 -4.2) (layer F.SilkS) hide
       (effects (font (size 1 1) (thickness 0.15)))
     )
@@
     (tags "test point SMD pad rectangle square")
     (attr virtual)
-    (fp_text reference J1 (at 0 -2.898) (layer F.SilkS)
+    (fp_text reference J1 (at 0 -2.898) (layer F.SilkS) hide
       (effects (font (size 1 1) (thickness 0.15)))
     )
@@
     (tags "test point SMD pad rectangle square")
     (attr virtual)
-    (fp_text reference J2 (at 0 -2.898) (layer F.SilkS)
+    (fp_text reference J2 (at 0 -2.898) (layer F.SilkS) hide
       (effects (font (size 1 1) (thickness 0.15)))
     )
@@
     (tags "resistor handsolder")
     (attr smd)
-    (fp_text reference R1 (at 0 -1.43 180) (layer F.SilkS)
-      (effects (font (size 1 1) (thickness 0.15)))
-    )
-    (fp_text value 4.7k (at 0 1.43 180) (layer F.Fab)
+    (fp_text reference R1 (at -2.7775 0.03 180) (layer F.SilkS)
+      (effects (font (size 1 1) (thickness 0.15)))
+    )
+    (fp_text value 4.7k (at 0 1.43 180) (layer F.SilkS) hide
       (effects (font (size 1 1) (thickness 0.15)))
     )
@@
     (tags "resistor handsolder")
     (attr smd)
-    (fp_text reference R2 (at 0 -1.43) (layer F.SilkS)
+    (fp_text reference R2 (at 3.0725 -0.05) (layer F.SilkS)
       (effects (font (size 1 1) (thickness 0.15)))
     )
@@
     (tags "resistor handsolder")
     (attr smd)
-    (fp_text reference R3 (at 0 -1.43 180) (layer F.SilkS)
+    (fp_text reference R3 (at 0 1.38 180) (layer F.SilkS)
       (effects (font (size 1 1) (thickness 0.15)))
     )
@@
     (descr "solder Pin_ with flat fork, hole diameter 0.7mm, length 6.5mm, width 1.8mm")
     (tags "solder Pin_ with flat fork")
-    (fp_text reference TP3 (at 0 1.8) (layer F.SilkS)
+    (fp_text reference TP3 (at 0.04 -2.01) (layer F.SilkS)
       (effects (font (size 1 1) (thickness 0.15)))
     )
@@
     (tags "capacitor handsolder")
     (attr smd)
-    (fp_text reference C4 (at 0 -1.43 270) (layer F.SilkS)
+    (fp_text reference C4 (at 2.6125 -0.03) (layer F.SilkS)
       (effects (font (size 1 1) (thickness 0.15)))
     )
@@
     )
   )
+  (gr_text "Current sensor v1.0-Allegro\n" (at 79.75 68.15) (layer B.SilkS)
+    (effects (font (size 1.3 1.3) (thickness 0.2)) (justify mirror))
+  )
+  (gr_text Vout (at 77.31 61.1) (layer F.SilkS)
+    (effects (font (size 1.5 1.5) (thickness 0.2)))
+  )
+  (gr_text GND (at 94.53 53.5) (layer F.SilkS)
+    (effects (font (size 1.5 1.5) (thickness 0.2)))
+  )
+  (gr_text CS (at 95.05 50.78) (layer F.SilkS)
+    (effects (font (size 1.5 1.5) (thickness 0.2)))
+  )
+  (gr_text "5V\n" (at 95.03 48.51) (layer F.SilkS)
+    (effects (font (size 1.5 1.5) (thickness 0.2)))
+  )
+  (gr_text 3 (at 96.93 55.44) (layer F.SilkS)
+    (effects (font (size 1 1) (thickness 0.1)))
+  )
+  (gr_text 1 (at 96.79 46.22) (layer F.SilkS)
+    (effects (font (size 1 1) (thickness 0.1)))
+  )
+  (gr_text CS (at 94.92 41.86) (layer F.SilkS)
+    (effects (font (size 1.5 1.5) (thickness 0.2)))
+  )
+  (gr_text GND (at 93.97 60.52) (layer F.SilkS)
+    (effects (font (size 1.5 1.5) (thickness 0.2)))
+  )
+  (gr_poly (pts (xy 62.55 51.98) (xy 63.43 51.99) (xy 63.01 52.49) (xy 62.97 52.49)) (layer F.SilkS) (width 0.15))
+  (gr_line (start 63 52.5) (end 63 52) (layer F.SilkS) (width 0.2))
+  (gr_line (start 62.5 52) (end 63 52.5) (layer F.SilkS) (width 0.2))
+  (gr_line (start 63.5 52) (end 62.5 52) (layer F.SilkS) (width 0.2))
+  (gr_line (start 63 52.5) (end 63.5 52) (layer F.SilkS) (width 0.2))
+  (gr_line (start 63 48.5) (end 63 52.5) (layer F.SilkS) (width 0.2))
   (gr_line (start 100 70) (end 100 30) (layer Edge.Cuts) (width 0.1))
   (gr_line (start 60 70) (end 100 70) (layer Edge.Cuts) (width 0.1))
@@
     (polygon
       (pts
-        (xy 60 51.25) (xy 68.5 51.125) (xy 68.5 59.875) (xy 60 60)
+        (xy 60 51.13) (xy 68.5 51.125) (xy 68.5 59.875) (xy 60 60)
       )
     )
